File: CPS3-OSCR.kicad_pcb (KiCad board)
At the start: 4 copper layers, 117.6 x 100 mm, 28 parts, among them J1 128MB, J2 64MB, J3 CART SLOT TOP ROW, J4 CART SLOT BOTTOM ROW, J5 5145154-1, J6 Conn_02x03_Counter_Clockwise, J7 Conn_02x03_Counter_Clockwise, M2_1 Screw_Terminal_01x01, M2_2 Screw_Terminal_01x01, M2_3 Screw_Terminal_01x01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

Commit message: Add voltage divider resitor to 3.3V and pullup's disable ic's as default
Parts:
- added R1: 10K, Resistor_SMD:R_0805_2012Metric, F.Cu at (112.7, 92.8)
- added R10: 2K, Resistor_SMD:R_0805_2012Metric, B.Cu at (126.6, 148.2)
- added R11: 2K, Resistor_SMD:R_0805_2012Metric, B.Cu at (124.6, 148.2)
- added R12: 2K, Resistor_SMD:R_0805_2012Metric, B.Cu at (122.6, 148.2)
- added R13: 2K, Resistor_SMD:R_0805_2012Metric, B.Cu at (177.4, 148.2)
- added R14: 2K, Resistor_SMD:R_0805_2012Metric, B.Cu at (175.4, 148.2)
- added R2: 10K, Resistor_SMD:R_0805_2012Metric, F.Cu at (115.3, 92.8)
- added R3: 10K, Resistor_SMD:R_0805_2012Metric, F.Cu at (125.4, 92.8)
- added R4: 10K, Resistor_SMD:R_0805_2012Metric, F.Cu at (178.8, 77.9)
- added R5: 1K, Resistor_SMD:R_0805_2012Metric, B.Cu at (126.6, 141.3)
- added R6: 1K, Resistor_SMD:R_0805_2012Metric, B.Cu at (124.6, 141.3)
- added R7: 1K, Resistor_SMD:R_0805_2012Metric, B.Cu at (122.6, 141.3)
- added R8: 1K, Resistor_SMD:R_0805_2012Metric, B.Cu at (177.4, 141.3)
- added R9: 1K, Resistor_SMD:R_0805_2012Metric, B.Cu at (175.4, 141.3)
- U1, U2, U3, U4: footprint Package_SO:SSOP-20_5.3x7.2mm_P0.65mm -> CPS3:SSOP-20_5.3x7.2mm_P0.65mm_.45
Connections:
- J6 pad 1: A23 -> /A23R
- J6 pad 2: unconnected-(J6-Pin_2-Pad2) -> /A23R
- J6 pad 3: A24 -> /A24R
- J6 pad 4: unconnected-(J6-Pin_4-Pad4) -> /A24R
- J6 pad 5: A25 -> /A25R
- J6 pad 6: unconnected-(J6-Pin_6-Pad6) -> /A25R
- J7 pad 1: A21 -> /A21R
- J7 pad 2: unconnected-(J7-Pin_2-Pad2) -> /A21R
- J7 pad 3: A22 -> /A22R
- J7 pad 4: unconnected-(J7-Pin_4-Pad4) -> /A22R
- J7 pad 5: A23 -> /A23R
- J7 pad 6: unconnected-(J7-Pin_6-Pad6) -> /A23R
- M2_5 pad 1: (no net) -> GND
Routing:
- net /A23R: track 0.00 -> 53.8 mm
- net A23: track 255.0 -> 206.4 mm, vias 1 -> 2
- net OE: track 258.5 -> 242.5 mm
- net BYTE: track 59.5 -> 48.7 mm
- net CE64LSB: track 81.4 -> 91.9 mm
- net CE128: track 20.0 -> 30.5 mm
- net CE64MSB: track 116.9 -> 127.4 mm
- net /A25R: track 0.00 -> 5.05 mm
- net /A24R: track 0.00 -> 5.05 mm
- net /A22R: track 0.00 -> 5.05 mm
- net /A21R: track 0.00 -> 5.05 mm
- net VCC: track 12.9 -> 17.2 mm, vias 5 -> 9
- net ~{CE}R_CST: track 25.4 -> 22.2 mm
- net A25: track 171.6 -> 169.7 mm, vias 2 -> 3
- net A24: track 187.6 -> 185.8 mm, vias 2 -> 3
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